Commit message: 10h44

File: urdf/Assem2.urdf (robot description, URDF)
Before this commit: robot Assem2, 7 links, 6 joints
Joints:
- joint joint_arm1: limit lower=-0.35 upper=0.35 effort=5 velocity=2 -> lower=-3.14 upper=3.14 effort=10 velocity=5
- joint joint_arm2: limit lower=-0.35 upper=0.35 effort=5 velocity=2 -> lower=-3.14 upper=3.14 effort=10 velocity=5
